Commit message: 增加控制器配置的注释

File: urdf/robot_cell.urdf.xacro (robot description, xacro)
@@ -1,33 +1,32 @@
 <?xml version="1.0"?>
-<robot xmlns:xacro="http://ros.org/wiki/xacro"
-       name="robot_cell" >
-  <!-- Robot Cell -->
-  <link name="robot_cell_link">
-    <inertial>
-      <origin xyz="0 0 0" rpy="0 0 0" />
-      <mass value="0.1"/>
-      <inertia ixx="1" ixy="0" ixz="0" iyy="1" iyz="0" izz="1" />
-    </inertial>
-    <visual>
-      <origin xyz="0 0 0" rpy="0 0 0" />
-      <geometry>
-        <mesh filename="package://macs_dual_arm/meshes/robot_cell/visual/robot_cell.dae"/>
-      </geometry>
-    </visual>
-    <collision>
-      <origin xyz = "0.6 0 -0.62" rpy="0 ${-pi/2} 0" />
-      <geometry>
-        <mesh filename="package://macs_dual_arm/meshes/robot_cell/collision/robot_cell_simplified.stl"
+<robot xmlns:xacro="http://ros.org/wiki/xacro" name="robot_cell">
+    <!-- Robot Cell -->
+    <link name="robot_cell_link">
+        <inertial>
+            <origin xyz="0 0 0" rpy="0 0 0" />
+            <mass value="0.1"/>
+            <inertia ixx="1" ixy="0" ixz="0" iyy="1" iyz="0" izz="1" />
+        </inertial>
+        <visual>
+            <origin xyz="0 0 0" rpy="0 0 0" />
+            <geometry>
+                <mesh filename="package://ordis_dual_arm/meshes/robot_cell/visual/robot_cell.dae"/>
+            </geometry>
+        </visual>
+        <collision>
+            <origin xyz = "0.6 0 -0.62" rpy="0 ${-pi/2} 0" />
+            <geometry>
+                <mesh filename="package://ordis_dual_arm/meshes/robot_cell/collision/robot_cell_simplified.stl"
         scale = "0.001 0.001 0.001"/>
-      </geometry>
-    </collision>
-  </link>
-  <!-- Used for fixing robot to Gazebo 'base_link' -->
-  <link name="world"/>
-  <!-- Robot Cell to World Joint -->
-  <joint name="fixed" type="fixed">
-    <origin xyz = "0 0 0" rpy="${pi/2} 0 0" />
-    <parent link="world"/>
-    <child link="robot_cell_link"/>
-  </joint>
+            </geometry>
+        </collision>
+    </link>
+    <!-- Used for fixing robot to Gazebo 'base_link' -->
+    <link name="world"/>
+    <!-- Robot Cell to World Joint -->
+    <joint name="fixed" type="fixed">
+        <origin xyz = "0 0 0" rpy="${pi/2} 0 0" />
+        <parent link="world"/>
+        <child link="robot_cell_link"/>
+    </joint>
 </robot>

File: urdf/ur5e_hande.urdf.xacro (robot description, xacro)
@@ -1,15 +1,14 @@
 <?xml version="1.0"?>
-<robot xmlns:xacro="http://ros.org/wiki/xacro"
-       name="ur5e_hande" >
-  <!-- UR5e robot -->
-  <xacro:include filename="$(find macs_dual_arm)/urdf/ur5e_robot.urdf.xacro" />
-  <!-- Hand-E gripper -->
-  <xacro:include filename="$(find hande_description)/urdf/robotiq_hande.urdf.xacro"/>
-  <xacro:robotiq_hande prefix=""/>
-  <!-- Connect Hand-E to UR5e arm-->
-  <joint name="arm_to_hand" type="fixed">
-    <parent link="wrist_3_link" />
-    <child link = "robotiq_hande_base_link" />
-    <origin xyz="0.0 0.0 0.0" rpy="0.0 0.0 0.0" />
-  </joint>
+<robot xmlns:xacro="http://ros.org/wiki/xacro" name="ur5e_hande">
+    <!-- UR5e robot -->
+    <xacro:include filename="$(find ordis_dual_arm)/urdf/ur5e_robot.urdf.xacro" />
+    <!-- Hand-E gripper -->
+    <xacro:include filename="$(find hande_description)/urdf/robotiq_hande.urdf.xacro"/>
+    <xacro:robotiq_hande prefix=""/>
+    <!-- Connect Hand-E to UR5e arm-->
+    <joint name="arm_to_hand" type="fixed">
+        <parent link="wrist_3_link" />
+        <child link = "robotiq_hande_base_link" />
+        <origin xyz="0.0 0.0 0.0" rpy="0.0 0.0 0.0" />
+    </joint>
 </robot>

File: urdf/ur5e_robot.urdf.xacro (robot description, xacro)
@@ -1,19 +1,16 @@
 <?xml version="1.0"?>
-<robot xmlns:xacro="http://ros.org/wiki/xacro"
-       name="ur5e" >
-  <!-- common stuff -->
-  <xacro:include filename="$(find ur5e_description)/urdf/common.gazebo.xacro" />
-  <!-- ur5e -->
-  <xacro:include filename="$(find macs_dual_arm)/urdf/ur5e.urdf.xacro" />
-  <!-- arm -->
-  <xacro:arg name="kinematics_config" default="$(find ur5e_description)/config/ur5e_default.yaml"/>
-  <xacro:ur5e_robot prefix="" joint_limited="false" use_effort_interface="true"
-    kinematics_file="${load_yaml('$(arg kinematics_config)')}"
-    />
-  <link name="world" />
-  <joint name="world_joint" type="fixed">
-    <parent link="world" />
-    <child link = "base_link" />
-    <origin xyz="0.0 0.0 0.0" rpy="0.0 0.0 0.0" />
-  </joint>
+<robot xmlns:xacro="http://ros.org/wiki/xacro" name="ur5e">
+    <!-- common stuff -->
+    <xacro:include filename="$(find ur5e_description)/urdf/common.gazebo.xacro" />
+    <!-- ur5e -->
+    <xacro:include filename="$(find ordis_dual_arm)/urdf/ur5e.urdf.xacro" />
+    <!-- arm -->
+    <xacro:arg name="kinematics_config" default="$(find ur5e_description)/config/ur5e_default.yaml"/>
+    <xacro:ur5e_robot prefix="" joint_limited="false" use_effort_interface="true" kinematics_file="${load_yaml('$(arg kinematics_config)')}" />
+    <link name="world" />
+    <joint name="world_joint" type="fixed">
+        <parent link="world" />
+        <child link = "base_link" />
+        <origin xyz="0.0 0.0 0.0" rpy="0.0 0.0 0.0" />
+    </joint>
 </robot>

File: urdf/ur5e_robot_joint_limited.urdf.xacro (robot description, xacro)
@@ -1,25 +1,16 @@
 <?xml version="1.0"?>
-<robot xmlns:xacro="http://ros.org/wiki/xacro"
-       name="ur5e" >
-  <!-- common stuff -->
-  <xacro:include filename="$(find ur5e_description)/urdf/common.gazebo.xacro" />
-  <!-- ur5e -->
-  <xacro:include filename="$(find macs_dual_arm)/urdf/ur5e.urdf.xacro" />
-  <!-- arm -->
-  <xacro:arg name="kinematics_config" default="$(find ur5e_description)/config/ur5e_default.yaml"/>
-  <xacro:ur5e_robot prefix="" joint_limited="true" use_effort_interface="true"
-    shoulder_pan_lower_limit="${-pi}" shoulder_pan_upper_limit="${pi}"
-    shoulder_lift_lower_limit="${-pi}" shoulder_lift_upper_limit="${pi}"
-    elbow_joint_lower_limit="${-pi}" elbow_joint_upper_limit="${pi}"
-    wrist_1_lower_limit="${-pi}" wrist_1_upper_limit="${pi}"
-    wrist_2_lower_limit="${-pi}" wrist_2_upper_limit="${pi}"
-    wrist_3_lower_limit="${-pi}" wrist_3_upper_limit="${pi}"
-    kinematics_file="${load_yaml('$(arg kinematics_config)')}"
-  />
-  <link name="world" />
-  <joint name="world_joint" type="fixed">
-    <parent link="world" />
-    <child link = "base_link" />
-    <origin xyz="0.0 0.0 0.0" rpy="0.0 0.0 0.0" />
-  </joint>
+<robot xmlns:xacro="http://ros.org/wiki/xacro" name="ur5e">
+    <!-- common stuff -->
+    <xacro:include filename="$(find ur5e_description)/urdf/common.gazebo.xacro" />
+    <!-- ur5e -->
+    <xacro:include filename="$(find ordis_dual_arm)/urdf/ur5e.urdf.xacro" />
+    <!-- arm -->
+    <xacro:arg name="kinematics_config" default="$(find ur5e_description)/config/ur5e_default.yaml"/>
+    <xacro:ur5e_robot prefix="" joint_limited="true" use_effort_interface="true" shoulder_pan_lower_limit="${-pi}" shoulder_pan_upper_limit="${pi}" shoulder_lift_lower_limit="${-pi}" shoulder_lift_upper_limit="${pi}" elbow_joint_lower_limit="${-pi}" elbow_joint_upper_limit="${pi}" wrist_1_lower_limit="${-pi}" wrist_1_upper_limit="${pi}" wrist_2_lower_limit="${-pi}" wrist_2_upper_limit="${pi}" wrist_3_lower_limit="${-pi}" wrist_3_upper_limit="${pi}" kinematics_file="${load_yaml('$(arg kinematics_config)')}" />
+    <link name="world" />
+    <joint name="world_joint" type="fixed">
+        <parent link="world" />
+        <child link = "base_link" />
+        <origin xyz="0.0 0.0 0.0" rpy="0.0 0.0 0.0" />
+    </joint>
 </robot>
